File: ice_cutter.kicad_sch (KiCad schematic)
At the start: 164 parts, among them J1 Conn_01x01_Male, J2 Barrel_Jack, J3 pot, J4 Conn_01x01_Male, J5 program, J6 program2, J7 hands, J8 UART, M1 Motor_Servo, M2 Motor_Servo, Q1 Q_PMOS_GSD, Q11 Q_NMOS_GSD, Q12 Q_NMOS_GSD, Q13 Q_NMOS_GSD, Q14 Q_NMOS_GSD, Q19 Q_PMOS_GSD, Q2 Q_PMOS_GSD, Q20 Q_PMOS_GSD, Q21 Q_PMOS_GSD, Q22 Q_PMOS_GSD, Q23 S8050_SMD, Q24 Q_NMOS_GSD, Q25 Q_PMOS_GSD, Q3 Q_PMOS_GSD, Q4 S8550, Q5 Q_NMOS_GSD, Q7 Q_NMOS_GSD, SW1 SW_Push, SW2 SW_Push, SW3 SW_Push, U1 LM358, U10 TMP117, U11 TM1620, U12 INA219AxD, U2 LM317_TO-252, U3 INA219AxD, U5 INA219AxD, U6 FJ4301AH, U7 FJ4301AH, U8 STM32G030XX, U9 SHT30-DIS

Commit message: 5V version - I hope it works
Parts:
- removed D2: 10V, Diode_SMD:D_SOD-123, symbol Device:D_Zener_Small
- added JP6: Jumper_2_Open, Jumper:SolderJumper-2_P1.3mm_Open_RoundedPad1.0x1.5mm, symbol Jumper:Jumper_2_Open
- added R67, R68, R69, R70, R71: 100R, Resistor_SMD:R_1206_3216Metric, symbol Device:R_Small_US
- R11, R3: value 15mR -> 12mR; LCSC C105381 -> C323773
- R17: value 4k7 -> 100R; footprint Resistor_SMD:R_0402_1005Metric -> Resistor_SMD:R_1206_3216Metric; LCSC C25900 -> C17901
Connections:
- net LV: now also U1.3 (+)
- net LV_Out: now also JP6.1 (A)
- net V_SS: no longer U1.3 (+)
- net Wire_H: now also R17.1, R67.1, R68.1; no longer R17.2
- net Wire_L: now also R69.2, R70.2, R71.2; no longer R17.1
- net at C10.1, JP2.1 (A), Q3.2 (S)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: now also JP6.2 (B)
- new net: R17.2, R67.2, R68.2, R69.1, R70.1, R71.1
Other:
- note added: "@12mR PGA /1 = 3.2A sense Range PGA /2 = 6.4A sense Range PGA /4 = 12.8A sense Range PGA /8 = 25A sense Range"
- note removed: "@15mR PGA /1 = 2.5A sense Range PGA /2 = 5A sense Range PGA /4 = 10A sense Range PGA /8 = 20A sense Range"
- moved on the sheet: C18, C19, C20, D3, D4, Q2, Q25, R20, R21, SW1, SW2, SW3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
