File: ice_cutter.kicad_pcb (KiCad board)
At the start: 4 copper layers, 90 x 100 mm, 194 parts, among them J1 Conn_01x01_Male, J2 Barrel_Jack, J3 pot, J4 Conn_01x01_Male, J5 program, J6 program2, J7 hands, J8 UART, M1 Motor_Servo, M2 Motor_Servo, Q1 Q_PMOS_GSD, Q10 S8050_SMD, Q11 Q_NMOS_GSD, Q12 Q_NMOS_GSD, Q13 Q_NMOS_GSD, Q14 Q_NMOS_GSD, Q15 S8550, Q16 S8050_SMD, Q17 S8050_SMD, Q18 S8050_SMD, Q19 Q_PMOS_GSD, Q2 Q_PMOS_GSD, Q20 Q_PMOS_GSD, Q21 Q_PMOS_GSD, Q22 Q_PMOS_GSD, Q23 S8050_SMD, Q24 Q_NMOS_GSD, Q25 Q_PMOS_GSD, Q3 Q_PMOS_GSD, Q4 S8550, Q5 Q_NMOS_GSD, Q6 S8550, Q7 Q_NMOS_GSD, Q8 S8050_SMD, Q9 S8050_SMD, SW1 SW_Push, SW2 SW_Push, SW3 SW_Push, U1 LM358, U10 TMP117, U11 TM1620, U12 INA219AxD, U2 LM317_TO-252, U3 INA219AxD, U5 INA219AxD, U6 FJ4301AH, U7 FJ4301AH, U8 STM32G030XX, U9 SHT30-DIS

Commit message: potential new version. Still to do Silkscreen and resistor value confirmations
Parts:
- moved TP22 42.6 mm to (135.4, 31.4)
- moved C22 19.4 mm to (126.8, 58.1), turned to 180 degrees
- moved Q24 17.4 mm to (151.7, 66.2), turned to -90 degrees
- moved U9 16.0 mm to (126.5, 60.7), turned to 90 degrees
- moved Q7 7.66 mm to (143.5, 66.4), turned to -90 degrees
- moved C26 6.86 mm to (151.2, 80.0)
- moved Q8 6.86 mm to (146.7, 77.4)
- moved R23 6.86 mm to (149.1, 81.9)
- moved R27 6.86 mm to (143.7, 81.5)
- moved R61 6.86 mm to (154.8, 76.3)
- moved C27 6.86 mm to (147.1, 79.9)
- moved Q10 6.86 mm to (146.7, 82.5)
- moved Q6 6.86 mm to (151.6, 77.4)
- moved Q9 6.86 mm to (151.6, 82.5)
- moved R19 6.86 mm to (149.1, 76.8)
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Connections:
- TP22 pad 1: /5V_SS -> /LV
- U1 pad 3: /5V_SS -> /V_SS
Routing:
- net VDC: track 63.5 -> 4.19 mm, vias 7 -> 41
- net /FET_GATE: track 11.2 -> 52.0 mm, vias 1 -> 14
- net /V_SS: track 140.0 -> 169.4 mm, vias 23 -> 31
- net /LV: track 53.5 -> 26.3 mm, vias 6 -> 76
- net /LV_Out: track 28.8 -> 49.6 mm
- net Net-(C10-Pad1): track 17.7 -> 30.1 mm, vias 4 -> 7
- net /Wire_L: track 28.3 -> 38.2 mm
- net +3V3: track 158.2 -> 166.8 mm, vias 19 -> 20
- net GND: track 188.0 -> 181.2 mm, vias 104 -> 219
- net /SCL: track 143.0 -> 149.7 mm
- net /5V_SS: track 6.29 -> 0.00 mm, vias 1 -> 0
- net Net-(R10-Pad2): track 0.00 -> 5.51 mm
- net Net-(U1-Pad2): track 3.36 -> 7.12 mm
- net /SDA: track 137.9 -> 141.3 mm, vias 7 -> 6
- net /Drive_FET: track 73.3 -> 71.0 mm
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- added copper zone on F.Cu, net /LV
- added copper zone on F.Cu, net VDC
Other:
- board text added: "Barrel_Jack"

Commit message: 5V version - I hope it works
Parts:
- removed D2: 10V, Diode_SMD:D_SOD-123
- added JP6: Jumper_2_Open, Jumper:SolderJumper-2_P1.3mm_Open_RoundedPad1.0x1.5mm, F.Cu at (100.4, 52.2)
- added R67: 100R, Resistor_SMD:R_1206_3216Metric, F.Cu at (146.4, 47.4)
- added R68: 100R, Resistor_SMD:R_1206_3216Metric, F.Cu at (148.9, 47.4)
- added R69: 100R, Resistor_SMD:R_1206_3216Metric, F.Cu at (156.4, 47.4)
- added R70: 100R, Resistor_SMD:R_1206_3216Metric, F.Cu at (153.9, 47.4)
- added R71: 100R, Resistor_SMD:R_1206_3216Metric, F.Cu at (151.4, 47.4)
- R11, R3: value 15mR -> 12mR
- R17: value 4k7 -> 100R; footprint Resistor_SMD:R_0402_1005Metric -> Resistor_SMD:R_1206_3216Metric
- moved R17 4.54 mm to (143.9, 47.4), turned to -90 degrees
Connections:
- R17 pad 1: /Wire_L -> /Wire_H
- R17 pad 2: /Wire_H -> Net-(R69-Pad1)
- U1 pad 3: /V_SS -> /LV
Routing:
- net Net-(R69-Pad1): track 0.00 -> 14.3 mm
- net /Wire_H: track 36.0 -> 23.2 mm
- net /SCL: track 149.7 -> 140.7 mm
- net /LV: track 26.3 -> 34.9 mm, vias 76 -> 79
- net /SDA: track 141.3 -> 134.2 mm, vias 6 -> 5
- net /V_SS: track 169.4 -> 162.7 mm
- net +3V3: track 166.8 -> 160.6 mm
- net Net-(C10-Pad1): track 30.1 -> 34.9 mm
- net GND: track 181.2 -> 178.2 mm, vias 219 -> 243
- net /Wire_L: track 38.2 -> 41.0 mm
- net /LV_Out: track 49.6 -> 52.1 mm
- net /FET_GATE: track 52.0 -> 50.2 mm
- net /FET_Drive1/Drive_Out: track 8.10 -> 7.34 mm
Other:
- board text added: "LV"

Commit message: havent saved again...
Changed lines of the file:
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@@
     (fp_line (start -1.6 -0.8) (end 1.6 -0.8) (layer "F.Fab") (width 0.1))
     (fp_line (start 1.6 0.8) (end -1.6 0.8) (layer "F.Fab") (width 0.1))
-    (pad "1" smd roundrect locked (at -1.4625 0 270) (size 1.125 1.75) (layers "F.Cu" "F.Paste" "F.Mask") (roundrect_rratio 0.222222)
+    (pad "1" smd roundrect locked (at -1.4625 0 270) (size 1.125 1.75) (layers "F.Cu" "F.Paste" "F.Mask") (roundrect_rratio 0.2222222222)
       (net 106 "Net-(R69-Pad1)") (pintype "passive"))
-    (pad "2" smd roundrect locked (at 1.4625 0 270) (size 1.125 1.75) (layers "F.Cu" "F.Paste" "F.Mask") (roundrect_rratio 0.222222)
+    (pad "2" smd roundrect locked (at 1.4625 0 270) (size 1.125 1.75) (layers "F.Cu" "F.Paste" "F.Mask") (roundrect_rratio 0.2222222222)
       (net 21 "/Wire_L") (pintype "passive"))
     (model "${KICAD6_3DMODEL_DIR}/Resistor_SMD.3dshapes/R_1206_3216Metric.wrl"
@@
     (fp_line (start -1.6 0.8) (end -1.6 -0.8) (layer "F.Fab") (width 0.1))
     (fp_line (start 1.6 -0.8) (end 1.6 0.8) (layer "F.Fab") (width 0.1))
-    (pad "1" smd roundrect locked (at -1.4625 0 270) (size 1.125 1.75) (layers "F.Cu" "F.Paste" "F.Mask") (roundrect_rratio 0.222222)
+    (pad "1" smd roundrect locked (at -1.4625 0 270) (size 1.125 1.75) (layers "F.Cu" "F.Paste" "F.Mask") (roundrect_rratio 0.2222222222)
       (net 19 "/Wire_H") (pintype "passive"))
-    (pad "2" smd roundrect locked (at 1.4625 0 270) (size 1.125 1.75) (layers "F.Cu" "F.Paste" "F.Mask") (roundrect_rratio 0.222222)
+    (pad "2" smd roundrect locked (at 1.4625 0 270) (size 1.125 1.75) (layers "F.Cu" "F.Paste" "F.Mask") (roundrect_rratio 0.2222222222)
       (net 106 "Net-(R69-Pad1)") (pintype "passive"))
     (model "${KICAD6_3DMODEL_DIR}/Resistor_SMD.3dshapes/R_1206_3216Metric.wrl"
@@
     (fp_line (start -1.6 0.8) (end -1.6 -0.8) (layer "F.Fab") (width 0.1))
     (fp_line (start 1.6 0.8) (end -1.6 0.8) (layer "F.Fab") (width 0.1))
-    (pad "1" smd roundrect locked (at -1.4625 0 270) (size 1.125 1.75) (layers "F.Cu" "F.Paste" "F.Mask") (roundrect_rratio 0.222222)
+    (pad "1" smd roundrect locked (at -1.4625 0 270) (size 1.125 1.75) (layers "F.Cu" "F.Paste" "F.Mask") (roundrect_rratio 0.2222222222)
       (net 106 "Net-(R69-Pad1)") (pintype "passive"))
-    (pad "2" smd roundrect locked (at 1.4625 0 270) (size 1.125 1.75) (layers "F.Cu" "F.Paste" "F.Mask") (roundrect_rratio 0.222222)
+    (pad "2" smd roundrect locked (at 1.4625 0 270) (size 1.125 1.75) (layers "F.Cu" "F.Paste" "F.Mask") (roundrect_rratio 0.2222222222)
       (net 21 "/Wire_L") (pintype "passive"))
     (model "${KICAD6_3DMODEL_DIR}/Resistor_SMD.3dshapes/R_1206_3216Metric.wrl"
@@
     (fp_line (start 1.6 0.8) (end -1.6 0.8) (layer "F.Fab") (width 0.1))
     (fp_line (start 1.6 -0.8) (end 1.6 0.8) (layer "F.Fab") (width 0.1))
-    (pad "1" smd roundrect locked (at -1.4625 0 270) (size 1.125 1.75) (layers "F.Cu" "F.Paste" "F.Mask") (roundrect_rratio 0.222222)
+    (pad "1" smd roundrect locked (at -1.4625 0 270) (size 1.125 1.75) (layers "F.Cu" "F.Paste" "F.Mask") (roundrect_rratio 0.2222222222)
       (net 19 "/Wire_H") (pintype "passive"))
-    (pad "2" smd roundrect locked (at 1.4625 0 270) (size 1.125 1.75) (layers "F.Cu" "F.Paste" "F.Mask") (roundrect_rratio 0.222222)
+    (pad "2" smd roundrect locked (at 1.4625 0 270) (size 1.125 1.75) (layers "F.Cu" "F.Paste" "F.Mask") (roundrect_rratio 0.2222222222)
       (net 106 "Net-(R69-Pad1)") (pintype "passive"))
     (model "${KICAD6_3DMODEL_DIR}/Resistor_SMD.3dshapes/R_1206_3216Metric.wrl"
@@
     (fp_line (start 3.15 -1.6) (end 3.15 1.6) (layer "F.Fab") (width 0.1))
     (fp_line (start 3.15 1.6) (end -3.15 1.6) (layer "F.Fab") (width 0.1))
-    (pad "1" smd roundrect locked (at -2.9625 0 270) (size 1.225 3.35) (layers "F.Cu" "F.Paste" "F.Mask") (roundrect_rratio 0.204082)
+    (pad "1" smd roundrect locked (at -2.9625 0 270) (size 1.225 3.35) (layers "F.Cu" "F.Paste" "F.Mask") (roundrect_rratio 0.2040816327)
       (net 99 "/LV_Out") (pintype "passive"))
-    (pad "2" smd roundrect locked (at 2.9625 0 270) (size 1.225 3.35) (layers "F.Cu" "F.Paste" "F.Mask") (roundrect_rratio 0.204082)
+    (pad "2" smd roundrect locked (at 2.9625 0 270) (size 1.225 3.35) (layers "F.Cu" "F.Paste" "F.Mask") (roundrect_rratio 0.2040816327)
       (net 97 "Net-(C10-Pad1)") (pintype "passive"))
     (model "${KICAD6_3DMODEL_DIR}/Resistor_SMD.3dshapes/R_2512_6332Metric.wrl"
@@
     (fp_line (start -1.6 -0.8) (end 1.6 -0.8) (layer "F.Fab") (width 0.1))
     (fp_line (start -1.6 0.8) (end -1.6 -0.8) (layer "F.Fab") (width 0.1))
-    (pad "1" smd roundrect locked (at -1.4625 0 270) (size 1.125 1.75) (layers "F.Cu" "F.Paste" "F.Mask") (roundrect_rratio 0.222222)
+    (pad "1" smd roundrect locked (at -1.4625 0 270) (size 1.125 1.75) (layers "F.Cu" "F.Paste" "F.Mask") (roundrect_rratio 0.2222222222)
       (net 106 "Net-(R69-Pad1)") (pintype "passive"))
-    (pad "2" smd roundrect locked (at 1.4625 0 270) (size 1.125 1.75) (layers "F.Cu" "F.Paste" "F.Mask") (roundrect_rratio 0.222222)
+    (pad "2" smd roundrect locked (at 1.4625 0 270) (size 1.125 1.75) (layers "F.Cu" "F.Paste" "F.Mask") (roundrect_rratio 0.2222222222)
       (net 21 "/Wire_L") (pintype "passive"))
     (model "${KICAD6_3DMODEL_DIR}/Resistor_SMD.3dshapes/R_1206_3216Metric.wrl"
@@
     (fp_line (start -1.6 0.8) (end -1.6 -0.8) (layer "F.Fab") (width 0.1))
     (fp_line (start 1.6 0.8) (end -1.6 0.8) (layer "F.Fab") (width 0.1))
-    (pad "1" smd roundrect locked (at -1.4625 0 270) (size 1.125 1.75) (layers "F.Cu" "F.Paste" "F.Mask") (roundrect_rratio 0.222222)
+    (pad "1" smd roundrect locked (at -1.4625 0 270) (size 1.125 1.75) (layers "F.Cu" "F.Paste" "F.Mask") (roundrect_rratio 0.2222222222)
       (net 19 "/Wire_H") (pintype "passive"))
-    (pad "2" smd roundrect locked (at 1.4625 0 270) (size 1.125 1.75) (layers "F.Cu" "F.Paste" "F.Mask") (roundrect_rratio 0.222222)
+    (pad "2" smd roundrect locked (at 1.4625 0 270) (size 1.125 1.75) (layers "F.Cu" "F.Paste" "F.Mask") (roundrect_rratio 0.2222222222)
       (net 106 "Net-(R69-Pad1)") (pintype "passive"))
     (model "${KICAD6_3DMODEL_DIR}/Resistor_SMD.3dshapes/R_1206_3216Metric.wrl"
